Commit message: update stl model, fix auto exposure bug and some small bugs

File: urdf/leadsense.urdf (robot description, URDF)
Before this commit: robot leadsense_camera, 3 links, 2 joints
Links:
- link leadsense_left_camera: geometry visual cylinder length=0.004 radius=0.007
- link leadsense_right_camera: geometry visual cylinder length=0.004 radius=0.007
Joints:
- joint leadsense_center_joint: origin xyz=0 -0.06 0 rpy=0 0 0 -> xyz=0 0 0 rpy=-1.57 0 -1.57

Commit message: Update to SDK 1.3.1. Add IMU topics, parameters, etc.

File: urdf/leadsense.urdf (robot description, URDF)
Before this commit: robot leadsense_camera, 3 links, 2 joints
Links:
- added link leadsense_imu_frame
Joints:
- added joint imu_link_joint: type fixed, parent leadsense_left_camera, child leadsense_imu_frame, origin xyz=0.09195 -0.00005 -0.009 rpy=0 0 0
- joint leadsense_center_joint: origin xyz=0 0 0 rpy=-1.57 0 -1.57 -> xyz=0 0 0 rpy=0 0 0
- joint leadsense_right_camera_joint: origin xyz=0 -0.12 0 rpy=0 0 0 -> xyz=0.12 0 0 rpy=0 0 0

Commit message: Update to 1.3.2: add new topics, add new parameters, fix timestamp bug.

File: urdf/leadsense.urdf (robot description, URDF)
Before this commit: robot leadsense_camera, 4 links, 3 joints
Links:
- added link leadsense_left_laser_scan_frame
Joints:
- added joint leadsense_left_laser_scan_frame_joint: type fixed, parent leadsense_left_camera, child leadsense_left_laser_scan_frame, origin xyz=0 0 0 rpy=-1.57 -1.57 0
